File: amp.kicad_sch (KiCad schematic)
At the start: 19 parts, among them J1 AudioJack3, J2 Conn_01x02_Socket, J3 Conn_01x02_Socket, J4 Conn_01x02_Socket, J5 Screw_Terminal_01x02, U1 TDA2030, U2 TDA2030, U3 TDA2030

Commit message: Add files via upload
Parts:
- added J6: Screw_Terminal_01x05, Package_QFP:EQFP-144-1EP_20x20mm_P0.5mm_EP5x5mm, symbol Connector:Screw_Terminal_01x05
Connections:
- net at C4.1, J1.S, J2.2 (Pin_2)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: now also J6.5 (Pin_5)
- net at J5.1 (Pin_1), U1.5 (+Vs), U2.5 (+Vs)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: now also J6.4 (Pin_4)
- net at J1.R, R1.1, RV2.3: now also J6.1 (Pin_1)
- net at J1.T, R2.1, RV3.3: now also J6.3 (Pin_3)
- net at R1.2, R2.2, RV1.3: now also J6.2 (Pin_2)
- no-connect marks 4 -> 3
Changed lines of the file:
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@@
+	)
+	(junction
+		(at 33.02 80.01)
+		(diameter 0)
+		(color 0 0 0 0)
+	)
+	(junction
+		(at 44.45 77.47)
+		(diameter 0)
+		(color 0 0 0 0)
 	)
 	(junction
@@
 	)
 	(junction
+		(at 20.32 55.88)
+		(diameter 0)
+		(color 0 0 0 0)
+	)
+	(junction
 		(at 71.12 45.72)
 		(diameter 0)
@@
 	)
 	(junction
+		(at 55.88 82.55)
+		(diameter 0)
+		(color 0 0 0 0)
+	)
+	(junction
 		(at 82.55 19.05)
 		(diameter 0)
@@
 	(junction
 		(at 82.55 36.83)
+		(diameter 0)
+		(color 0 0 0 0)
+	)
+	(junction
+		(at 63.5 53.34)
 		(diameter 0)
 		(color 0 0 0 0)
@@
 	)
 	(no_connect
-		(at 68.58 87.63)
-	)
-	(no_connect
 		(at 82.55 24.13)
 	)
@@
 	(wire
 		(pts
+			(xy 63.5 87.63) (xy 63.5 53.34)
+		)
+		(stroke
+			(width 0)
+			(type default)
+		)
+	)
+	(wire
+		(pts
 			(xy 67.31 49.53) (xy 87.63 49.53)
 		)
@@
 	(wire
 		(pts
+			(xy 55.88 82.55) (xy 92.71 82.55)
+		)
+		(stroke
+			(width 0)
+			(type default)
+		)
+	)
+	(wire
+		(pts
+			(xy 92.71 87.63) (xy 63.5 87.63)
+		)
+		(stroke
+			(width 0)
+			(type default)
+		)
+	)
+	(wire
+		(pts
 			(xy 30.48 26.67) (xy 43.18 26.67)
 		)
@@
 	(wire
 		(pts
+			(xy 33.02 80.01) (xy 92.71 80.01)
+		)
+		(stroke
+			(width 0)
+			(type default)
+		)
+	)
+	(wire
+		(pts
 			(xy 29.21 78.74) (xy 29.21 63.5)
 		)
@@
 	(wire
 		(pts
+			(xy 44.45 77.47) (xy 44.45 82.55)
+		)
+		(stroke
+			(width 0)
+			(type default)
+		)
+	)
+	(wire
+		(pts
 			(xy 76.2 64.77) (xy 76.2 72.39)
 		)
@@
 	(wire
 		(pts
+			(xy 63.5 53.34) (xy 71.12 53.34)
+		)
+		(stroke
+			(width 0)
+			(type default)
+		)
+	)
+	(wire
+		(pts
+			(xy 44.45 77.47) (xy 92.71 77.47)
+		)
+		(stroke
+			(width 0)
+			(type default)
+		)
+	)
+	(wire
+		(pts
 			(xy 19.05 53.34) (xy 21.59 53.34)
 		)
@@
 	(wire
 		(pts
+			(xy 92.71 85.09) (xy 20.32 85.09)
+		)
+		(stroke
+			(width 0)
+			(type default)
+		)
+	)
+	(wire
+		(pts
 			(xy 25.4 71.12) (xy 36.83 71.12)
 		)
@@
 	(wire
 		(pts
-			(xy 33.02 68.58) (xy 33.02 82.55)
+			(xy 33.02 68.58) (xy 33.02 80.01)
 		)
 		(stroke
@@
 	(wire
 		(pts
-			(xy 19.05 55.88) (xy 67.31 55.88)
+			(xy 19.05 55.88) (xy 20.32 55.88)
 		)
 		(stroke
@@
 	(wire
 		(pts
+			(xy 20.32 85.09) (xy 20.32 55.88)
+		)
+		(stroke
+			(width 0)
+			(type default)
+		)
+	)
+	(wire
+		(pts
 			(xy 95.25 19.05) (xy 82.55 19.05)
 		)
@@
 	(wire
 		(pts
-			(xy 21.59 53.34) (xy 71.12 53.34)
+			(xy 21.59 53.34) (xy 63.5 53.34)
 		)
 		(stroke
@@
 	(wire
 		(pts
+			(xy 20.32 55.88) (xy 67.31 55.88)
+		)
+		(stroke
+			(width 0)
+			(type default)
+		)
+	)
+	(wire
+		(pts
 			(xy 52.07 72.39) (xy 52.07 78.74)
 		)
@@
 	(wire
 		(pts
-			(xy 44.45 73.66) (xy 44.45 82.55)
+			(xy 44.45 73.66) (xy 44.45 77.47)
 		)
 		(stroke
@@
 		(pts
 			(xy 44.45 54.61) (xy 44.45 57.15)
+		)
+		(stroke
+			(width 0)
+			(type default)
+		)
+	)
+	(wire
+		(pts
+			(xy 33.02 80.01) (xy 33.02 82.55)
 		)
 		(stroke
@@
 					(unit 1)
 				)
+			)
+		)
+	)
+	(symbol
+		(lib_id "Connector:Screw_Terminal_01x05")
+		(at 97.79 82.55 0)
+		(unit 1)
+		(body_style 1)
+		(exclude_from_sim no)
+		(in_bom yes)
+		(on_board yes)
+		(in_pos_files yes)
+		(dnp no)
+		(property "Reference" "J6"
+			(at 100.33 81.2799 0)
+			(show_name no)
+			(do_not_autoplace no)
+			(effects
+				(font
+					(size 1.27 1.27)
+				)
+				(justify left)
+			)
+		)
+		(property "Value" "Screw_Terminal_01x05"
+			(at 100.33 83.8199 0)
+			(show_name no)
+			(do_not_autoplace no)
+			(effects
+				(font
+					(size 1.27 1.27)
+				)
+				(justify left)
+			)
+		)
+		(property "Footprint" "Package_QFP:EQFP-144-1EP_20x20mm_P0.5mm_EP5x5mm"
+			(at 97.79 82.55 0)
+			(hide yes)
+			(show_name no)
+			(do_not_autoplace no)
+			(effects
+				(font
+					(size 1.27 1.27)
+				)
+			)
+		)
+		(property "Datasheet" ""
+			(at 97.79 82.55 0)
+			(hide yes)
+			(show_name no)
+			(do_not_autoplace no)
+			(effects
+				(font
+					(size 1.27 1.27)
+				)
+			)
+		)
+		(property "Description" "Generic screw terminal, single row, 01x05, script generated (kicad-library-utils/schlib/autogen/connector/)"
+			(at 97.79 82.55 0)
+			(hide yes)
+			(show_name no)
+			(do_not_autoplace no)
+			(effects
+				(font
+					(size 1.27 1.27)
+				)
+			)
+		)
+		(pin "4"
+		)
+		(pin "2"
+		)
+		(pin "5"
+		)
+		(pin "1"
+		)
+		(pin "3"
+		)
+		(instances
+			(project "amp"
+				(path "/77d9bcae-62d9-40fa-8a3e-f215d2f400a3"
+					(reference "J6")
+					(unit 1)
+				)
