File: amp.kicad_pcb (KiCad board)
At the start: 2 copper layers, 99.5 x 75 mm, 19 parts, among them J1 AudioJack3, J2 Conn_01x02_Socket, J3 Conn_01x02_Socket, J4 Conn_01x02_Socket, J5 Screw_Terminal_01x02, U1 TDA2030, U2 TDA2030, U3 TDA2030

Commit message: Add files via upload
Parts:
- added gnd: Screw_Terminal_01x05, TerminalBlock_Phoenix:TerminalBlock_Phoenix_MKDS-1,5-5_1x05_P5.00mm_Horizontal, F.Cu at (35.0, 72.0)
- J2, J3: value Conn_01x02_Socket -> pitch
- J4: value Conn_01x02_Socket -> subwoofer
- J5: value Screw_Terminal_01x02 -> Screw_Terminal
- L1: value L -> passive filter
- RV1, RV2, RV3: value R_Potentiometer -> Potentiometer
Routing:
- net Net-(J6-Pin_2): track 137.8 -> 241.4 mm
- net Net-(J6-Pin_1): track 160.0 -> 249.8 mm
- net Net-(J5-Pin_1): track 110.6 -> 198.3 mm
- net Net-(J2-Pin_2): track 259.0 -> 297.4 mm
- net Net-(J6-Pin_3): track 165.5 -> 194.9 mm
Other:
- board text added: "ring"
- board text added: "sub"
- board text added: "tip"

Commit message: Add files via upload
Other:
- outline, holes or cut-outs redrawn
- board text added: "-"
Changed lines of the file:
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@@
 			(layer "F.Fab")
 		)
-		(fp_text user "${REFERENCE}"
-			(at 2.5 3.2 90)
+		(fp_text user "-"
+			(at 5 5.5 90)
 			(layer "F.Fab")
 			(effects
@@
 		(layer "Edge.Cuts")
 	)
+	(gr_circle
+		(center 29 70)
+		(end 29 68)
+		(stroke
+			(width 0.05)
+			(type default)
+		)
+		(fill no)
+		(layer "Edge.Cuts")
+	)
+	(gr_circle
+		(center 30 20)
+		(end 30 18)
+		(stroke
+			(width 0.05)
+			(type default)
+		)
+		(fill no)
+		(layer "Edge.Cuts")
+	)
+	(gr_circle
+		(center 105 20)
+		(end 105 22)
+		(stroke
+			(width 0.05)
+			(type default)
+		)
+		(fill no)
+		(layer "Edge.Cuts")
+	)
 	(gr_text "ring"
 		(at 35 77.5 0)
@@
 		)
 	)
+	(gr_text "-"
+		(at 12.5 50 90)
+		(layer "F.Fab")
+		(effects
+			(font
+				(size 1 1)
+				(thickness 0.15)
+			)
+		)
+	)
+	(gr_text "-"
+		(at 12.5 63.5 90)
+		(layer "F.Fab")
+		(effects
+			(font
+				(size 1 1)
+				(thickness 0.15)
+			)
+		)
+	)
+	(gr_text "-"
+		(at 12.5 77 90)
+		(layer "F.Fab")
+		(effects
+			(font
+				(size 1 1)
+				(thickness 0.15)
+			)
+		)
+	)
 	(segment
 		(start 84.3875 28.662779)
@@
 	)
 	(segment
-		(start 46.324452 57.638048)
-		(end 63.3 40.6625)
-		(width 1.2)
-		(layer "F.Cu")
-		(net "Net-(J3-Pin_1)")
-	)
-	(segment
-		(start 19.361952 57.638048)
-		(end 46.324452 57.638048)
-		(width 1.2)
-		(layer "F.Cu")
-		(net "Net-(J3-Pin_1)")
-	)
-	(segment
-		(start 63.3 40.6625)
-		(end 63.3 29.5)
-		(width 1.2)
-		(layer "F.Cu")
-		(net "Net-(J3-Pin_1)")
-	)
-	(segment
-		(start 18.5 58.5)
-		(end 19.361952 57.638048)
-		(width 1.2)
-		(layer "F.Cu")
-		(net "Net-(J3-Pin_1)")
-	)
-	(segment
-		(start 84.5 32.5)
-		(end 96.275 32.5)
-		(width 0.7)
-		(layer "B.Cu")
-		(net "Net-(C3-Pad1)")
-	)
-	(segment
-		(start 96.275 32.5)
-		(end 97.775 31)
-		(width 0.7)
-		(layer "B.Cu")
-		(net "Net-(C3-Pad1)")
-	)
-	(segment
-		(start 65.5 51.5)
-		(end 84.5 32.5)
-		(width 0.7)
-		(layer "B.Cu")
-		(net "Net-(C3-Pad1)")
-	)
-	(segment
-		(start 40.135 48.295)
-		(end 24.205 48.295)
-		(width 0.4)
-		(layer "F.Cu")
-		(net "Net-(J6-Pin_1)")
-	)
-	(segment
-		(start 15.5 61)
-		(end 16 61.5)
-		(width 0.4)
-		(layer "F.Cu")
-		(net "Net-(J6-Pin_1)")
-	)
-	(segment
-		(start 39.5 67.5)
-		(end 100.5 67.5)
-		(width 0.6)
-		(layer "F.Cu")
-		(net "Net-(J6-Pin_1)")
-	)
-	(segment
-		(start 15.5 57)
-		(end 15.5 61)
-		(width 0.4)
-		(layer "F.Cu")
-		(net "Net-(J6-Pin_1)")
-	)
-	(segment
-		(start 16 61.5)
-		(end 84.25 61.5)
-		(width 0.4)
-		(layer "F.Cu")
-		(net "Net-(J6-Pin_1)")
-	)
-	(segment
-		(start 102.5 52.25)
-		(end 98 47.75)
-		(width 0.6)
-		(layer "F.Cu")
-		(net "Net-(J6-Pin_1)")
-	)
-	(segment
-		(start 35 72)
-		(end 39.5 67.5)
-		(width 0.6)
-		(layer "F.Cu")
-		(net "Net-(J6-Pin_1)")
-	)
-	(segment
-		(start 100.5 67.5)
-		(end 102.5 65.5)
-		(width 0.6)
-		(layer "F.Cu")
-		(net "Net-(J6-Pin_1)")
-	)
-	(segment
-		(start 24.205 48.295)
-		(end 15.5 57)
-		(width 0.4)
-		(layer "F.Cu")
-		(net "Net-(J6-Pin_1)")
-	)
-	(segment
-		(start 102.5 65.5)
-		(end 102.5 52.25)
-		(width 0.6)
-		(layer "F.Cu")
-		(net "Net-(J6-Pin_1)")
-	)
-	(segment
-		(start 84.25 61.5)
-		(end 98 47.75)
-		(width 0.4)
-		(layer "F.Cu")
-		(net "Net-(J6-Pin_1)")
-	)
-	(segment
-		(start 38.99 47.15)
-		(end 40.135 48.295)
-		(width 0.4)
-		(layer "B.Cu")
-		(net "Net-(J6-Pin_1)")
-	)
-	(segment
-		(start 22 16.5)
-		(end 38.99 33.49)
-		(width 0.4)
-		(layer "B.Cu")
-		(net "Net-(J6-Pin_1)")
-	)
-	(segment
-		(start 38.99 33.49)
-		(end 38.99 47.15)
-		(width 0.4)
-		(layer "B.Cu")
-		(net "Net-(J6-Pin_1)")
-	)
-	(segment
 		(start 45 72)
 		(end 41.5 75.5)
@@
 	)
 	(segment
+		(start 40.135 48.295)
+		(end 24.205 48.295)
+		(width 0.4)
+		(layer "F.Cu")
+		(net "Net-(J6-Pin_1)")
+	)
+	(segment
+		(start 15.5 61)
+		(end 16 61.5)
+		(width 0.4)
+		(layer "F.Cu")
+		(net "Net-(J6-Pin_1)")
+	)
+	(segment
+		(start 39.5 67.5)
+		(end 100.5 67.5)
+		(width 0.6)
+		(layer "F.Cu")
+		(net "Net-(J6-Pin_1)")
+	)
+	(segment
+		(start 15.5 57)
+		(end 15.5 61)
+		(width 0.4)
+		(layer "F.Cu")
+		(net "Net-(J6-Pin_1)")
+	)
+	(segment
+		(start 16 61.5)
+		(end 84.25 61.5)
+		(width 0.4)
+		(layer "F.Cu")
+		(net "Net-(J6-Pin_1)")
+	)
+	(segment
+		(start 102.5 52.25)
+		(end 98 47.75)
+		(width 0.6)
+		(layer "F.Cu")
+		(net "Net-(J6-Pin_1)")
+	)
+	(segment
+		(start 35 72)
+		(end 39.5 67.5)
+		(width 0.6)
+		(layer "F.Cu")
+		(net "Net-(J6-Pin_1)")
+	)
+	(segment
+		(start 100.5 67.5)
+		(end 102.5 65.5)
+		(width 0.6)
+		(layer "F.Cu")
+		(net "Net-(J6-Pin_1)")
+	)
+	(segment
+		(start 24.205 48.295)
+		(end 15.5 57)
+		(width 0.4)
+		(layer "F.Cu")
+		(net "Net-(J6-Pin_1)")
+	)
+	(segment
+		(start 102.5 65.5)
+		(end 102.5 52.25)
+		(width 0.6)
+		(layer "F.Cu")
+		(net "Net-(J6-Pin_1)")
+	)
+	(segment
+		(start 84.25 61.5)
+		(end 98 47.75)
+		(width 0.4)
+		(layer "F.Cu")
+		(net "Net-(J6-Pin_1)")
+	)
+	(segment
+		(start 38.99 47.15)
+		(end 40.135 48.295)
+		(width 0.4)
+		(layer "B.Cu")
+		(net "Net-(J6-Pin_1)")
+	)
+	(segment
+		(start 22 16.5)
+		(end 38.99 33.49)
+		(width 0.4)
+		(layer "B.Cu")
+		(net "Net-(J6-Pin_1)")
+	)
+	(segment
+		(start 38.99 33.49)
+		(end 38.99 47.15)
+		(width 0.4)
+		(layer "B.Cu")
+		(net "Net-(J6-Pin_1)")
+	)
+	(segment
 		(start 102 33.5)
 		(end 98 33.5)
@@
 		(net "Net-(J6-Pin_2)")
 	)
+	(segment
+		(start 46.324452 57.638048)
+		(end 63.3 40.6625)
+		(width 1.2)
+		(layer "F.Cu")
+		(net "Net-(J3-Pin_1)")
+	)
+	(segment
+		(start 19.361952 57.638048)
+		(end 46.324452 57.638048)
+		(width 1.2)
+		(layer "F.Cu")
+		(net "Net-(J3-Pin_1)")
+	)
+	(segment
+		(start 63.3 40.6625)
+		(end 63.3 29.5)
+		(width 1.2)
+		(layer "F.Cu")
+		(net "Net-(J3-Pin_1)")
+	)
+	(segment
+		(start 18.5 58.5)
+		(end 19.361952 57.638048)
+		(width 1.2)
+		(layer "F.Cu")
+		(net "Net-(J3-Pin_1)")
+	)
+	(segment
+		(start 84.5 32.5)
+		(end 96.275 32.5)
+		(width 0.7)
+		(layer "B.Cu")
+		(net "Net-(C3-Pad1)")
+	)
+	(segment
+		(start 96.275 32.5)
+		(end 97.775 31)
+		(width 0.7)
+		(layer "B.Cu")
+		(net "Net-(C3-Pad1)")
+	)
+	(segment
+		(start 65.5 51.5)
+		(end 84.5 32.5)
+		(width 0.7)
+		(layer "B.Cu")
+		(net "Net-(C3-Pad1)")
+	)
 	(embedded_fonts no)
