File: amp/amp.kicad_pcb (KiCad board)
At the start: 2 copper layers, 100 x 99 mm, 53 parts, among them J1 AudioJack3, J2 Conn_01x02_Socket, J3 Conn_01x02_Socket, J4 Conn_01x02_Socket, J5 Screw_Terminal_01x02, J6 Screw_Terminal_01x05, U1 TDA2030, U2 TDA2030, U3 TDA2030

Commit message: Add files via upload
Parts:
- added REF**: MountingHole_3.2mm_M3, MountingHole:MountingHole_3.2mm_M3, F.Cu at (32.0, 31.5)
- J2: value Conn_01x02_Socket -> speaker L
- J3: value Conn_01x02_Socket -> speaker R
- J4: value Conn_01x02_Socket -> subwoofer
- J5: value Screw_Terminal_01x02 -> 16V
- J6: value Screw_Terminal_01x05 -> debug port
- moved J1 1.50 mm to (19.0, 104.5)
Routing:
- net Net-(D3-A): track 324.2 -> 231.6 mm
- net Net-(J6-Pin_3): track 254.1 -> 188.1 mm
- net Net-(D1-K): track 363.8 -> 361.2 mm
- net Net-(U3--): track 159.2 -> 158.0 mm
- net Net-(J6-Pin_1): track 238.1 -> 238.7 mm
Other:
- outline, holes or cut-outs redrawn
- board text added: "+"
- board text added: "-"
- board text added: "ring"
- board text added: "sub"
- board text added: "tip"
